File: minix-keyboard.kicad_pcb (KiCad board)
At the start: 2 copper layers, 254 x 104.8 mm, 126 parts, among them J1 AVR-ISP-6, SW1 SW_Push, U1 ATmega32U4-AU, U2 PRTR5V0U2X, Y1 16MHz

Commit message: Add promicro header
Parts:
- added U3: ProMicro-keebio, Keebio-Parts:ArduinoProMicro-TopSide, B.Cu at (41.9, 33.1)
- moved D1 2.29 mm to (41.3, 35.8)
- moved D2 2.28 mm to (60.3, 35.8)
Connections:
- J1 pad 1: MISO -> COL10
- J1 pad 3: SCK -> COL9
- J1 pad 4: MOSI -> COL11
- U1 pad 1: Net-(U1-Pad1) -> COL3
- U1 pad 10: MOSI -> COL11
- U1 pad 11: MISO -> COL10
- U1 pad 18: Net-(U1-Pad18) -> ROW0
- U1 pad 25: Net-(U1-Pad25) -> COL0
- U1 pad 27: Net-(U1-Pad27) -> COL2
- U1 pad 28: Net-(U1-Pad28) -> COL4
- U1 pad 29: Net-(U1-Pad29) -> COL5
- U1 pad 30: Net-(U1-Pad30) -> COL12
- U1 pad 31: Net-(U1-Pad31) -> COL1
- U1 pad 36: Net-(U1-Pad36) -> COL8
- U1 pad 37: Net-(U1-Pad37) -> COL7
- U1 pad 38: Net-(U1-Pad38) -> COL6
- U1 pad 9: SCK -> COL9
Routing:
- net ROW0: track 0.00 -> 243.5 mm, vias 0 -> 1
- net Net-(D1-Pad2): track 12.6 -> 10.3 mm
- net Net-(D2-Pad2): track 12.6 -> 10.3 mm

Commit message: Update schematic
Connections:
- J1 pad 1: COL10 -> COL8
- J1 pad 4: COL11 -> COL7
- U1 pad 10: COL11 -> COL7
- U1 pad 11: COL10 -> COL8
- U1 pad 30: COL12 -> COL6
- U1 pad 36: COL8 -> COL10
- U1 pad 37: COL7 -> COL11
- U1 pad 38: COL6 -> COL12
- U3 pad 13: COL12 -> COL6
- U3 pad 14: COL11 -> COL7
- U3 pad 15: COL10 -> COL8
- U3 pad 17: COL8 -> COL10
- U3 pad 18: COL7 -> COL11
- U3 pad 19: COL6 -> COL12
Routing:
- net COL5: track 0.00 -> 71.8 mm
- net COL4: track 0.00 -> 55.9 mm
- net COL3: track 0.00 -> 41.9 mm
- net COL2: track 0.00 -> 22.3 mm
- net COL0: track 0.00 -> 15.9 mm
- net ROW0: track 243.5 -> 230.0 mm, vias 1 -> 0
- net COL1: track 0.00 -> 6.51 mm

Commit message: Routing switches
Routing:
- net COL11: track 0.00 -> 275.8 mm
- net COL10: track 0.00 -> 250.8 mm
- net COL9: track 0.00 -> 227.9 mm
- net COL12: track 0.00 -> 224.8 mm
- net ROW1: track 0.00 -> 219.1 mm
- net ROW2: track 0.00 -> 211.0 mm
- net ROW0: track 230.0 -> 439.3 mm, vias 0 -> 2
- net ROW3: track 0.00 -> 204.5 mm
- net COL8: track 0.00 -> 181.0 mm
- net COL6: track 0.00 -> 156.8 mm
- net COL7: track 0.00 -> 115.7 mm
- net COL3: track 41.9 -> 109.9 mm
- net COL0: track 15.9 -> 77.8 mm
- net COL5: track 71.8 -> 115.9 mm
- net COL4: track 55.9 -> 99.9 mm
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